Commit message: custom symmetry command probability set

File: resources/go2w/urdf/go2w_d435i.urdf (robot description, URDF)
Before this commit: robot go2w_description, 35 links, 34 joints
Joints:
- joint front_camera_joint: origin xyz=0.32715 -0.00003 0.04297 rpy=0 0 0 -> xyz=0.354 -0.00003 0.018 rpy=0 0 0

Commit message: camera encoder

File: resources/go2w/urdf/go2w_d435i.urdf (robot description, URDF)
Before this commit: robot go2w_description, 35 links, 34 joints
Links:
- link FL_foot: geometry collision cylinder length=0.045 radius=0.087; visual mesh filename=package://go2w/meshes/left_wheel.dae
- link FR_foot: geometry collision cylinder length=0.045 radius=0.087; visual mesh filename=package://go2w/meshes/right_wheel.dae
- link RL_foot: geometry collision cylinder length=0.045 radius=0.087; visual mesh filename=package://go2w/meshes/left_wheel.dae
- link RR_foot: geometry collision cylinder length=0.045 radius=0.087; visual mesh filename=package://go2w/meshes/right_wheel.dae

File: resources/go2w/urdf/go2w_description.urdf (robot description, URDF)
Before this commit: robot go2w_description, 33 links, 32 joints
Links:
- link FL_foot: geometry collision cylinder length=0.045 radius=0.087; visual mesh filename=package://go2w/meshes/left_wheel.dae
- link FR_foot: geometry collision cylinder length=0.045 radius=0.087; visual mesh filename=package://go2w/meshes/right_wheel.dae
- link RL_foot: geometry collision cylinder length=0.045 radius=0.087; visual mesh filename=package://go2w/meshes/left_wheel.dae
- link RR_foot: geometry collision cylinder length=0.045 radius=0.087; visual mesh filename=package://go2w/meshes/right_wheel.dae
